File: RGB-IR Backlight 7x7/Electrical/7x7RGB-IR-J010129B.sch (EAGLE design)
At the start: 457 parts, among them P4 CON2X3, Q1 NPN_DUAL, Q10 NPN_DUAL, Q11 NPN_DUAL, Q12 NPN_DUAL, Q2 NPN_DUAL, Q3 NPN_DUAL, Q4 NPN_DUAL, Q5 NPN_DUAL, Q6 NPN_DUAL, Q7 NPN_DUAL, Q8 NPN_DUAL, Q9 NPN_DUAL, U1 AP8802, U2 AP8802, U3 AP8802, U4 AP8802

Commit message: Add 7x7 RGB files
Add current PCB and cable assembly files for 7x7 RGB panel
Parts:
- removed RGB1, RGB10, RGB11, RGB12, RGB13, RGB14, RGB15, RGB16, RGB17, RGB18, RGB19, RGB2, RGB20, RGB21, RGB22, RGB23, RGB24, RGB25, RGB26, RGB27, RGB28, RGB29, RGB3, RGB30, RGB31, RGB32, RGB33, RGB34, RGB35, RGB36, RGB37, RGB38, RGB39, RGB4, RGB40, RGB41, RGB42, RGB43, RGB44, RGB45, RGB46, RGB47, RGB48, RGB49, RGB5, RGB50, RGB51, RGB52, RGB53, RGB54, RGB55, RGB56, RGB57, RGB58, RGB59, RGB6, RGB60, RGB61, RGB62, RGB63, RGB64, RGB7, RGB8, RGB9: LED_RGB_PADSUNPLUS, STEVES_BU:LED_RGB_PADSUNPLUS
- added BLU1, BLU10, BLU11, BLU12, BLU13, BLU14, BLU15, BLU16, BLU17, BLU18, BLU19, BLU2, BLU20, BLU21, BLU22, BLU23, BLU24, BLU25, BLU26, BLU27, BLU28, BLU29, BLU3, BLU30, BLU31, BLU32, BLU33, BLU34, BLU35, BLU36, BLU37, BLU38, BLU39, BLU4, BLU40, BLU41, BLU42, BLU43, BLU44, BLU45, BLU46, BLU47, BLU48, BLU49, BLU5, BLU50, BLU51, BLU52, BLU53, BLU54, BLU55, BLU56, BLU57, BLU58, BLU59, BLU6, BLU60, BLU61, BLU62, BLU63, BLU64, BLU7, BLU8, BLU9: SP-BLU, RGB_IR_J010131revC:LED-TH
- added GRN1, GRN10, GRN11, GRN12, GRN13, GRN14, GRN15, GRN16, GRN17, GRN18, GRN19, GRN2, GRN20, GRN21, GRN22, GRN23, GRN24, GRN25, GRN26, GRN27, GRN28, GRN29, GRN3, GRN30, GRN31, GRN32, GRN33, GRN34, GRN35, GRN36, GRN37, GRN38, GRN39, GRN4, GRN40, GRN41, GRN42, GRN43, GRN44, GRN45, GRN46, GRN47, GRN48, GRN49, GRN5, GRN50, GRN51, GRN52, GRN53, GRN54, GRN55, GRN56, GRN57, GRN58, GRN59, GRN6, GRN60, GRN61, GRN62, GRN63, GRN64, GRN7, GRN8, GRN9: SP-GRN, RGB_IR_J010131revC:LED-TH
- added RED1, RED10, RED11, RED12, RED13, RED14, RED15, RED16, RED17, RED18, RED19, RED2, RED20, RED21, RED22, RED23, RED24, RED25, RED26, RED27, RED28, RED29, RED3, RED30, RED31, RED32, RED33, RED34, RED35, RED36, RED37, RED38, RED39, RED4, RED40, RED41, RED42, RED43, RED44, RED45, RED46, RED47, RED48, RED49, RED5, RED50, RED51, RED52, RED53, RED54, RED55, RED56, RED57, RED58, RED59, RED6, RED60, RED61, RED62, RED63, RED64, RED7, RED8, RED9: SP-RED, RGB_IR_J010131revC:LED-TH
- R17, R21: value (none) -> 0R0
- R18, R52: device resistor:R-US_R1206 -> STEVES_BU:RESISTOR_SM1206S
Connections:
- removed net N$343: C6.2, D114.K, D130.K, D81.K, D98.K, R21.2, RGB24.PAD, RGB32.PAD
- removed net N$413: RGB60.RA, RGB61.RC
- removed net N$417: RGB57.BA, RGB58.BC
- removed net N$418: RGB58.BA, RGB59.BC
- removed net N$419: RGB59.BA, RGB60.BC
- removed net N$420: RGB60.BA, RGB61.BC
- removed net N$421: RGB61.BA, RGB62.BC
- removed net N$422: RGB62.BA, RGB63.BC
- new net IR_RET2: BLU24.TH, BLU32.TH, C6.2, D114.K, D130.K, D81.K, D98.K, GRN24.TH, GRN32.TH, R21.2, RED24.TH, RED32.TH
- new net N$262: RED34.A, RED35.K
- new net N$267: RED33.A, RED34.K
- new net N$28: GRN5.A, GRN6.K
- new net N$292: BLU33.A, BLU34.K
- new net N$357: GRN46.A, GRN47.K
- new net N$403: RED61.A, RED62.K
- new net N$410: BLU59.A, BLU60.K
- net BLU1K: now also BLU1.K; no longer RGB1.BC
- net BLU1K2: now also BLU9.K; no longer RGB9.BC
- net BLU2K1: now also BLU17.K; no longer RGB17.BC
- net BLU2K2: now also BLU25.K; no longer RGB25.BC
- net BLU3K: now also BLU33.K; no longer RGB33.BC
- net GRN1K: now also GRN1.K; no longer RGB1.GC
- net GRN1K2: now also GRN9.K; no longer RGB9.GC
- net GRN2K1: now also GRN17.K; no longer RGB17.GC
- net GRN2K2: now also GRN25.K; no longer RGB25.GC
- net GRN3K: now also GRN33.K; no longer RGB33.GC
- net GULA_1: now also GRN57.K; no longer RGB57.GC
- net GULA_2: now also RED57.K; no longer RGB57.RC
- net GULA_3: now also GRN41.K; no longer RGB41.GC
- net GULA_4: now also RED41.K; no longer RGB41.RC
- net HS1: now also BLU2.TH, BLU3.TH, BLU4.TH, BLU5.TH, BLU6.TH, BLU7.TH, GRN2.TH, GRN3.TH, GRN4.TH, GRN5.TH, GRN6.TH, GRN7.TH, RED2.TH, RED3.TH, RED4.TH, RED5.TH, RED6.TH, RED7.TH; no longer RGB2.PAD, RGB3.PAD, RGB4.PAD, RGB5.PAD, RGB6.PAD, RGB7.PAD
- net HS2: now also BLU10.TH, BLU11.TH, BLU12.TH, BLU13.TH, BLU14.TH, BLU15.TH, GRN10.TH, GRN11.TH, GRN12.TH, GRN13.TH, GRN14.TH, GRN15.TH, RED10.TH, RED11.TH, RED12.TH, RED13.TH, RED14.TH, RED15.TH; no longer RGB10.PAD, RGB11.PAD, RGB12.PAD, RGB13.PAD, RGB14.PAD, RGB15.PAD
- net HS3: now also BLU18.TH, BLU19.TH, BLU20.TH, BLU21.TH, BLU22.TH, BLU23.TH, GRN18.TH, GRN19.TH, GRN20.TH, GRN21.TH, GRN22.TH, GRN23.TH, RED18.TH, RED19.TH, RED20.TH, RED21.TH, RED22.TH, RED23.TH; no longer RGB18.PAD, RGB19.PAD, RGB20.PAD, RGB21.PAD, RGB22.PAD, RGB23.PAD
- net HS4: now also BLU26.TH, BLU27.TH, BLU28.TH, BLU29.TH, BLU30.TH, BLU31.TH, GRN26.TH, GRN27.TH, GRN28.TH, GRN29.TH, GRN30.TH, GRN31.TH, RED26.TH, RED27.TH, RED28.TH, RED29.TH, RED30.TH, RED31.TH; no longer RGB26.PAD, RGB27.PAD, RGB28.PAD, RGB29.PAD, RGB30.PAD, RGB31.PAD
- net HS5: now also BLU34.TH, BLU35.TH, BLU36.TH, BLU37.TH, BLU38.TH, BLU39.TH, GRN34.TH, GRN35.TH, GRN36.TH, GRN37.TH, GRN38.TH, GRN39.TH, RED34.TH, RED35.TH, RED36.TH, RED37.TH, RED38.TH, RED39.TH; no longer RGB34.PAD, RGB35.PAD, RGB36.PAD, RGB37.PAD, RGB38.PAD, RGB39.PAD
- net HS6: now also BLU42.TH, BLU43.TH, BLU44.TH, BLU45.TH, BLU46.TH, BLU47.TH, GRN42.TH, GRN43.TH, GRN44.TH, GRN45.TH, GRN46.TH, GRN47.TH, RED42.TH, RED43.TH, RED44.TH, RED45.TH, RED46.TH, RED47.TH; no longer RGB42.PAD, RGB43.PAD, RGB44.PAD, RGB45.PAD, RGB46.PAD, RGB47.PAD
- net HS7: now also BLU50.TH, BLU51.TH, BLU52.TH, BLU53.TH, BLU54.TH, BLU55.TH, GRN50.TH, GRN51.TH, GRN52.TH, GRN53.TH, GRN54.TH, GRN55.TH, RED50.TH, RED51.TH, RED52.TH, RED53.TH, RED54.TH, RED55.TH; no longer RGB50.PAD, RGB51.PAD, RGB52.PAD, RGB53.PAD, RGB54.PAD, RGB55.PAD
- net HS8: now also BLU58.TH, BLU59.TH, BLU60.TH, BLU61.TH, BLU62.TH, BLU63.TH, GRN58.TH, GRN59.TH, GRN60.TH, GRN61.TH, GRN62.TH, GRN63.TH, RED58.TH, RED59.TH, RED60.TH, RED61.TH, RED62.TH, RED63.TH; no longer RGB58.PAD, RGB59.PAD, RGB60.PAD, RGB61.PAD, RGB62.PAD, RGB63.PAD
- net IR_DRV3: now also BLU33.TH, BLU41.TH, GRN33.TH, GRN41.TH, RED33.TH, RED41.TH; no longer RGB33.PAD, RGB41.PAD
- net IR_DRV4: now also BLU49.TH, BLU57.TH, GRN49.TH, GRN57.TH, RED49.TH, RED57.TH; no longer RGB49.PAD, RGB57.PAD
- net IR_DRV_UL1: now also BLU1.TH, BLU9.TH, GRN1.TH, GRN9.TH, RED1.TH, RED9.TH; no longer RGB1.PAD, RGB9.PAD
- net IR_DRV_UL2: now also BLU17.TH, BLU25.TH, GRN17.TH, GRN25.TH, RED17.TH, RED25.TH; no longer RGB17.PAD, RGB25.PAD
- net IR_RET3: now also BLU40.TH, BLU48.TH, GRN40.TH, GRN48.TH, RED40.TH, RED48.TH; no longer RGB40.PAD, RGB48.PAD
- net IR_RET_UL1: now also BLU16.TH, BLU8.TH, GRN16.TH, GRN8.TH, RED16.TH, RED8.TH; no longer RGB16.PAD, RGB8.PAD
- net I_RET4: now also BLU56.TH, BLU64.TH, GRN56.TH, GRN64.TH, RED56.TH, RED64.TH; no longer RGB56.PAD, RGB64.PAD
- net N$1: now also GRN10.A, GRN11.K; no longer RGB15.GA, RGB16.GC
- net N$100: now also BLU23.A, BLU24.K; no longer RGB17.RA, RGB18.RC
- net N$101: now also BLU19.A, BLU20.K; no longer RGB17.BA, RGB18.BC
- net N$102: now also RED19.A, RED20.K; no longer RGB18.BA, RGB19.BC
- net N$103: now also GRN19.A, GRN20.K; no longer RGB19.BA, RGB20.BC
- net N$104: now also GRN26.A, GRN27.K; no longer RGB20.BA, RGB21.BC
- net N$105: now also BLU22.A, BLU23.K; no longer RGB21.BA, RGB22.BC
- net N$106: now also RED22.A, RED23.K; no longer RGB22.BA, RGB23.BC
- net N$107: now also GRN22.A, GRN23.K; no longer RGB23.BA, RGB24.BC
- net N$12: now also RED10.A, RED11.K; no longer RGB13.GA, RGB14.GC
- net N$13: now also RED10.K, RED9.A; no longer RGB12.GA, RGB13.GC
- net N$135: now also GRN4.A, GRN5.K; no longer RGB7.GA, RGB8.GC
- net N$136: now also RED5.A, RED6.K; no longer RGB6.GA, RGB7.GC
- net N$137: now also RED4.A, RED5.K; no longer RGB5.GA, RGB6.GC
- net N$138: now also BLU4.A, BLU5.K; no longer RGB4.GA, RGB5.GC
- net N$139: now also BLU5.A, BLU6.K; no longer RGB3.GA, RGB4.GC
- net N$140: now also GRN2.A, GRN3.K; no longer RGB2.GA, RGB3.GC
- net N$141: now also GRN1.A, GRN2.K; no longer RGB1.GA, RGB2.GC
- net N$142: now also GRN7.A, GRN8.K; no longer RGB7.RA, RGB8.RC
- net N$143: now also RED7.A, RED8.K; no longer RGB6.RA, RGB7.RC
- net N$144: now also BLU7.A, BLU8.K; no longer RGB5.RA, RGB6.RC
- net N$145: now also BLU3.A, BLU4.K; no longer RGB4.RA, RGB5.RC
- net N$146: now also RED3.A, RED4.K; no longer RGB3.RA, RGB4.RC
- net N$147: now also RED2.A, RED3.K; no longer RGB2.RA, RGB3.RC
- net N$148: now also RED1.A, RED2.K; no longer RGB1.RA, RGB2.RC
- net N$149: now also BLU1.A, BLU2.K; no longer RGB1.BA, RGB2.BC
- net N$150: now also BLU2.A, BLU3.K; no longer RGB2.BA, RGB3.BC
- net N$151: now also GRN3.A, GRN4.K; no longer RGB3.BA, RGB4.BC
- net N$152: now also GRN14.A, GRN15.K; no longer RGB4.BA, RGB5.BC
- net N$153: now also BLU6.A, BLU7.K; no longer RGB5.BA, RGB6.BC
- net N$154: now also RED6.A, RED7.K; no longer RGB6.BA, RGB7.BC
- net N$155: now also GRN6.A, GRN7.K; no longer RGB7.BA, RGB8.BC
- net N$177: now also GRN41.A, GRN42.K; no longer RGB46.GA, RGB47.GC
- net N$178: now also RED42.A, RED43.K; no longer RGB45.GA, RGB46.GC
- net N$179: now also RED41.A, RED42.K; no longer RGB44.GA, RGB45.GC
- net N$181: now also BLU41.A, BLU42.K; no longer RGB43.GA, RGB44.GC
- net N$188: now also BLU42.A, BLU43.K; no longer RGB42.GA, RGB43.GC
- net N$190: now also RED58.A, RED59.K; no longer RGB63.GA, RGB64.GC
- net N$191: now also GRN25.A, GRN26.K; no longer RGB31.GA, RGB32.GC
- net N$192: now also RED26.A, RED27.K; no longer RGB30.GA, RGB31.GC
- net N$193: now also RED25.A, RED26.K; no longer RGB29.GA, RGB30.GC
- net N$194: now also BLU25.A, BLU26.K; no longer RGB28.GA, RGB29.GC
- net N$195: now also BLU26.A, BLU27.K; no longer RGB27.GA, RGB28.GC
- net N$196: now also GRN29.A, GRN30.K; no longer RGB26.GA, RGB27.GC
- net N$197: now also GRN28.A, GRN29.K; no longer RGB25.GA, RGB26.GC
- net N$198: now also RED29.A, RED30.K; no longer RGB31.RA, RGB32.RC
- net N$199: now also RED28.A, RED29.K; no longer RGB30.RA, RGB31.RC
- net N$20: now also RED49.K; no longer RGB49.RC
- net N$200: now also BLU28.A, BLU29.K; no longer RGB29.RA, RGB30.RC
- net N$201: now also BLU29.A, BLU30.K; no longer RGB28.RA, RGB29.RC
- net N$202: now also GRN31.A, GRN32.K; no longer RGB27.RA, RGB28.RC
- net N$203: now also RED31.A, RED32.K; no longer RGB26.RA, RGB27.RC
- net N$204: now also BLU31.A, BLU32.K; no longer RGB25.RA, RGB26.RC
- net N$205: now also BLU27.A, BLU28.K; no longer RGB25.BA, RGB26.BC
- net N$206: now also RED27.A, RED28.K; no longer RGB26.BA, RGB27.BC
- net N$207: now also GRN27.A, GRN28.K; no longer RGB27.BA, RGB28.BC
- net N$208: now also GRN34.A, GRN35.K; no longer RGB28.BA, RGB29.BC
- net N$209: now also BLU30.A, BLU31.K; no longer RGB29.BA, RGB30.BC
- net N$210: now also RED30.A, RED31.K; no longer RGB30.BA, RGB31.BC
- net N$211: now also GRN30.A, GRN31.K; no longer RGB31.BA, RGB32.BC
- net N$230: now also GRN45.A, GRN46.K; no longer RGB41.GA, RGB42.GC
- net N$233: now also GRN44.A, GRN45.K; no longer RGB47.RA, RGB48.RC
- net N$235: now also RED45.A, RED46.K; no longer RGB46.RA, RGB47.RC
- net N$238: now also RED44.A, RED45.K; no longer RGB45.RA, RGB46.RC
- net N$239: now also BLU44.A, BLU45.K; no longer RGB44.RA, RGB45.RC
- net N$240: now also BLU45.A, BLU46.K; no longer RGB43.RA, RGB44.RC
- net N$241: now also GRN47.A, GRN48.K; no longer RGB42.RA, RGB43.RC
- net N$242: now also RED47.A, RED48.K; no longer RGB41.RA, RGB42.RC
- net N$243: now also BLU47.A, BLU48.K; no longer RGB41.BA, RGB42.BC
- net N$244: now also BLU43.A, BLU44.K; no longer RGB42.BA, RGB43.BC
- net N$245: now also RED43.A, RED44.K; no longer RGB43.BA, RGB44.BC
- net N$248: now also GRN43.A, GRN44.K; no longer RGB44.BA, RGB45.BC
- net N$249: now also GRN50.A, GRN51.K; no longer RGB45.BA, RGB46.BC
- net N$250: now also BLU46.A, BLU47.K; no longer RGB46.BA, RGB47.BC
- net N$251: now also RED46.A, RED47.K; no longer RGB47.BA, RGB48.BC
- net N$26: now also GRN58.A, GRN59.K; no longer RGB63.BA, RGB64.BC
- net N$261: now also GRN33.A, GRN34.K; no longer RGB33.RA, RGB34.RC
- net N$294: now also GRN49.A, GRN50.K; no longer RGB55.GA, RGB56.GC
- net N$295: now also RED50.A, RED51.K; no longer RGB54.GA, RGB55.GC
- net N$296: now also RED49.A, RED50.K; no longer RGB53.GA, RGB54.GC
- net N$297: now also BLU49.A, BLU50.K; no longer RGB52.GA, RGB53.GC
- net N$298: now also BLU50.A, BLU51.K; no longer RGB51.GA, RGB52.GC
- net N$299: now also GRN53.A, GRN54.K; no longer RGB50.GA, RGB51.GC
- net N$30: now also GRN57.A, GRN58.K; no longer RGB63.RA, RGB64.RC
- net N$300: now also GRN52.A, GRN53.K; no longer RGB49.GA, RGB50.GC
- net N$301: now also RED53.A, RED54.K; no longer RGB55.RA, RGB56.RC
- net N$302: now also RED52.A, RED53.K; no longer RGB54.RA, RGB55.RC
- net N$303: now also BLU52.A, BLU53.K; no longer RGB53.RA, RGB54.RC
- net N$304: now also BLU53.A, BLU54.K; no longer RGB52.RA, RGB53.RC
- net N$305: now also GRN55.A, GRN56.K; no longer RGB51.RA, RGB52.RC
- net N$306: now also RED55.A, RED56.K; no longer RGB50.RA, RGB51.RC
- net N$307: now also BLU55.A, BLU56.K; no longer RGB49.RA, RGB50.RC
- net N$308: now also BLU51.A, BLU52.K; no longer RGB49.BA, RGB50.BC
- net N$309: now also RED51.A, RED52.K; no longer RGB50.BA, RGB51.BC
- net N$310: now also GRN51.A, GRN52.K; no longer RGB51.BA, RGB52.BC
- net N$311: now also RED57.A, RED58.K; no longer RGB52.BA, RGB53.BC
- net N$312: now also BLU54.A, BLU55.K; no longer RGB53.BA, RGB54.BC
- net N$313: now also RED54.A, RED55.K; no longer RGB54.BA, RGB55.BC
- net N$314: now also GRN54.A, GRN55.K; no longer RGB55.BA, RGB56.BC
- net N$344: now also BLU34.A, BLU35.K; no longer RGB39.GA, RGB40.GC
- net N$345: now also GRN37.A, GRN38.K; no longer RGB38.GA, RGB39.GC
- net N$346: now also GRN36.A, GRN37.K; no longer RGB37.GA, RGB38.GC
- net N$347: now also RED37.A, RED38.K; no longer RGB36.GA, RGB37.GC
- net N$348: now also RED36.A, RED37.K; no longer RGB35.GA, RGB36.GC
- net N$349: now also BLU36.A, BLU37.K; no longer RGB34.GA, RGB35.GC
- net N$350: now also BLU37.A, BLU38.K; no longer RGB33.GA, RGB34.GC
- net N$351: now also GRN39.A, GRN40.K; no longer RGB39.RA, RGB40.RC
- net N$352: now also RED39.A, RED40.K; no longer RGB38.RA, RGB39.RC
- net N$353: now also BLU39.A, BLU40.K; no longer RGB37.RA, RGB38.RC
- net N$354: now also BLU35.A, BLU36.K; no longer RGB36.RA, RGB37.RC
- net N$355: now also RED35.A, RED36.K; no longer RGB35.RA, RGB36.RC
- net N$356: now also GRN35.A, GRN36.K; no longer RGB34.RA, RGB35.RC
- net N$358: now also BLU38.A, BLU39.K; no longer RGB33.BA, RGB34.BC
- net N$359: now also RED38.A, RED39.K; no longer RGB34.BA, RGB35.BC
- net N$360: now also GRN38.A, GRN39.K; no longer RGB35.BA, RGB36.BC
- net N$361: now also BLU57.A, BLU58.K; no longer RGB36.BA, RGB37.BC
- net N$362: now also BLU58.A, BLU59.K; no longer RGB37.BA, RGB38.BC
- net N$363: now also GRN61.A, GRN62.K; no longer RGB38.BA, RGB39.BC
- net N$364: now also GRN60.A, GRN61.K; no longer RGB39.BA, RGB40.BC
- net N$40: now also BLU10.K, BLU9.A; no longer RGB11.GA, RGB12.GC
- net N$401: now also BLU41.K; no longer RGB41.BC
- net N$404: now also RED60.A, RED61.K; no longer RGB62.GA, RGB63.GC
- net N$405: now also BLU60.A, BLU61.K; no longer RGB61.GA, RGB62.GC
- net N$406: now also BLU61.A, BLU62.K; no longer RGB60.GA, RGB61.GC
- net N$407: now also GRN63.A, GRN64.K; no longer RGB59.GA, RGB60.GC
- net N$408: now also RED63.A, RED64.K; no longer RGB58.GA, RGB59.GC
- net N$409: now also BLU63.A, BLU64.K; no longer RGB57.GA, RGB58.GC
- net N$41: now also BLU10.A, BLU11.K; no longer RGB10.GA, RGB11.GC
- net N$411: now also RED59.A, RED60.K; no longer RGB62.RA, RGB63.RC
- net N$412: now also GRN59.A, GRN60.K; no longer RGB61.RA, RGB62.RC
- net N$414: now also BLU62.A, BLU63.K; no longer RGB59.RA, RGB60.RC
- net N$415: now also RED62.A, RED63.K; no longer RGB58.RA, RGB59.RC
- net N$416: now also GRN62.A, GRN63.K; no longer RGB57.RA, RGB58.RC
- net N$42: now also GRN13.A, GRN14.K; no longer RGB10.GC, RGB9.GA
- net N$43: now also GRN12.A, GRN13.K; no longer RGB15.RA, RGB16.RC
- net N$44: now also RED13.A, RED14.K; no longer RGB14.RA, RGB15.RC
- net N$45: now also RED12.A, RED13.K; no longer RGB13.RA, RGB14.RC
- net N$46: now also BLU12.A, BLU13.K; no longer RGB12.RA, RGB13.RC
- net N$47: now also BLU13.A, BLU14.K; no longer RGB11.RA, RGB12.RC
- net N$48: now also GRN15.A, GRN16.K; no longer RGB10.RA, RGB11.RC
- net N$49: now also RED15.A, RED16.K; no longer RGB10.RC, RGB9.RA
- net N$5: now also GRN49.K; no longer RGB49.GC
- net N$50: now also BLU15.A, BLU16.K; no longer RGB10.BC, RGB9.BA
- net N$51: now also BLU11.A, BLU12.K; no longer RGB10.BA, RGB11.BC
- net N$52: now also RED11.A, RED12.K; no longer RGB11.BA, RGB12.BC
- net N$53: now also GRN11.A, GRN12.K; no longer RGB12.BA, RGB13.BC
- net N$54: now also GRN18.A, GRN19.K; no longer RGB13.BA, RGB14.BC
- net N$55: now also BLU14.A, BLU15.K; no longer RGB14.BA, RGB15.BC
- net N$56: now also RED14.A, RED15.K; no longer RGB15.BA, RGB16.BC
- net N$6: now also BLU49.K; no longer RGB49.BC
- net N$7: now also GRN10.K, GRN9.A; no longer RGB14.GA, RGB15.GC
- net N$8: now also BLU57.K; no longer RGB57.BC
- net N$86: now also GRN17.A, GRN18.K; no longer RGB23.GA, RGB24.GC
- net N$87: now also RED18.A, RED19.K; no longer RGB22.GA, RGB23.GC
- net N$88: now also RED17.A, RED18.K; no longer RGB21.GA, RGB22.GC
- net N$89: now also BLU17.A, BLU18.K; no longer RGB20.GA, RGB21.GC
- net N$90: now also BLU18.A, BLU19.K; no longer RGB19.GA, RGB20.GC
- net N$91: now also GRN21.A, GRN22.K; no longer RGB18.GA, RGB19.GC
- net N$92: now also GRN20.A, GRN21.K; no longer RGB17.GA, RGB18.GC
- net N$93: now also RED21.A, RED22.K; no longer RGB23.RA, RGB24.RC
- net N$94: now also RED20.A, RED21.K; no longer RGB22.RA, RGB23.RC
- net N$95: now also BLU20.A, BLU21.K; no longer RGB21.RA, RGB22.RC
- net N$96: now also BLU21.A, BLU22.K; no longer RGB20.RA, RGB21.RC
- net N$97: now also GRN42.A, GRN43.K; no longer RGB47.GA, RGB48.GC
- net N$98: now also GRN23.A, GRN24.K; no longer RGB19.RA, RGB20.RC
- net N$99: now also RED23.A, RED24.K; no longer RGB18.RA, RGB19.RC
- net RED1K: now also RED1.K; no longer RGB1.RC
- net RED1K2: now also RED9.K; no longer RGB9.RC
- net RED2K1: now also RED17.K; no longer RGB17.RC
- net RED2K2: now also RED25.K; no longer RGB25.RC
- net RED3K: now also RED33.K; no longer RGB33.RC
- net V_RGB: now also BLU16.A, BLU24.A, BLU32.A, BLU40.A, BLU48.A, BLU56.A, BLU64.A, BLU8.A, GRN16.A, GRN24.A, GRN32.A, GRN40.A, GRN48.A, GRN56.A, GRN64.A, GRN8.A, RED16.A, RED24.A, RED32.A, RED40.A, RED48.A, RED56.A, RED64.A, RED8.A; no longer RGB16.BA, RGB16.GA, RGB16.RA, RGB24.BA, RGB24.GA, RGB24.RA, RGB32.BA, RGB32.GA, RGB32.RA, RGB40.BA, RGB40.GA, RGB40.RA, RGB48.BA, RGB48.GA, RGB48.RA, RGB56.BA, RGB56.GA, RGB56.RA, RGB64.BA, RGB64.GA, RGB64.RA, RGB8.BA, RGB8.GA, RGB8.RA
Other:
- note added: "TODO - seperate out RGB footprint into 3 separate for CircuitHub"
- note removed: "TODO: - Connect IGND to POWER IN not ribbon - Connect LGND to ribbon ground - make IGND tracks bigger - two grounds on each ribbon?"
